File: AmbientCN3791.kicad_sch (KiCad schematic)
At the start: 56 parts, among them J1 Conn_01x02, J2 Conn_01x02, J3 Conn_01x02, J4 Conn_01x04, J5 Conn_01x04, J7 Conn_01x02, J8 Conn_01x02, Q1 AO3401A, Q2 AO3401A, U1 CN3791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

Commit message: WIP: 0.5
Parts:
- C6, C9: LCSC C307331 -> C1525
Changed lines of the file:
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@@
 	(title_block
 		(title "AmbientCN3791")
-		(date "2025-07-15")
-		(rev "v0.3")
+		(date "2026-03-11")
+		(rev "v0.5")
 		(company "//piernov")
 	)
@@
 			)
 		)
+		(property "Sim.Pins" "1=K 2=A"
+			(at 111.76 67.31 0)
+			(effects
+				(font
+					(size 1.27 1.27)
+				)
+				(hide yes)
+			)
+		)
 		(pin "1"
 		)
@@
 			)
 		)
-		(property "LCSC" "C307331"
+		(property "LCSC" "C1525"
 			(at 71.12 129.54 0)
 			(effects
@@
 	)
 	(symbol
+		(lib_name "LED_Small_1")
 		(lib_id "Device:LED_Small")
 		(at 111.76 64.77 180)
@@
 			)
 		)
+		(property "Sim.Pins" "1=K 2=A"
+			(at 111.76 64.77 0)
+			(effects
+				(font
+					(size 1.27 1.27)
+				)
+				(hide yes)
+			)
+		)
 		(pin "1"
 		)
@@
 			)
 		)
-		(property "LCSC" "C307331"
+		(property "LCSC" "C1525"
 			(at 189.23 57.15 0)
 			(effects

Commit message: WIP2
Parts:
- removed RV1: 20k, Potentiometer_SMD:Potentiometer_Bourns_3224J_Horizontal, symbol Device:R_Potentiometer_Trim
- added RV1: 200k, Potentiometer_SMD:Potentiometer_Bourns_3314J_Vertical, symbol Device:R_Potentiometer
- J3: footprint Connector_JST:JST_XH_S2B-XH-A_1x02_P2.50mm_Horizontal -> Connector_PinSocket_2.54mm:PinSocket_1x02_P2.54mm_Vertical
- R1: value 100k -> 33k; LCSC C25741 -> C25779
- R2: value 10k -> 12k; LCSC C25744 -> C25752
Connections:
- net GND: now also R2.2
- net at R2.1, U1.6 (MPPT): now also RV1.1; no longer R1.2
- new net: R1.2, RV1.2
Other:
- moved on the sheet: C1, C12, C13, C5, C7, J1, R1, R11, R2, R22

Commit message: WIP3
Parts:
- D3, D4: value PMEG6030EP,115 -> PMEG6030ELPX; LCSC C456127 -> C2908821
- L1: value 47µF/3A -> 47µH/3A
- RV1: FT Rotation Offset (none) -> -90
Changed lines of the file:
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@@
 			)
 		)
-		(property "Value" "47µF/3A"
+		(property "Value" "47µH/3A"
 			(at 153.67 39.37 90)
 			(effects
@@
 		(property "LCSC" "C124643"
 			(at 92.71 63.5 90)
+			(effects
+				(font
+					(size 1.27 1.27)
+				)
+				(hide yes)
+			)
+		)
+		(property "FT Rotation Offset" "-90"
+			(at 92.71 63.5 0)
 			(effects
 				(font
@@
 			)
 		)
-		(property "Value" "PMEG6030EP,115"
+		(property "Value" "PMEG6030ELPX"
 			(at 170.942 24.384 90)
 			(effects
@@
 			)
 		)
-		(property "LCSC" "C456127"
+		(property "LCSC" "C2908821"
 			(at 171.45 41.91 90)
 			(effects
@@
 			)
 		)
-		(property "Value" "PMEG6030EP,115"
+		(property "Value" "PMEG6030ELPX"
 			(at 147.32 50.8 90)
 			(effects
@@
 			)
 		)
-		(property "LCSC" "C456127"
+		(property "LCSC" "C2908821"
 			(at 147.32 57.15 90)
 			(effects

Commit message: Fix opamp supply polarity + KiCad 10 upgrade
Parts:
- D3, D4: footprint PCM_Diode_SMD_AKL:D_SOD-128 -> Diode_SMD:D_SOD-128
