File: AudioPowerBoard.kicad_sch (KiCad schematic)
At the start: 4 parts

Commit message: Update
Other:
- sheet AmbienCN3791 renamed AmbientCN3791
Changed lines of the file:
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@@
 			(color 0 0 0 0.0000)
 		)
-		(property "Sheetname" "AmbienCN3791"
+		(property "Sheetname" "AmbientCN3791"
 			(at 53.34 52.6284 0)
 			(effects

Commit message: Update
Parts:
- H1, H2, H3, H4: now not fitted
Changed lines of the file:
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@@
 		(exclude_from_sim no)
 		(in_bom no)
-		(on_board yes)
-		(dnp no)
+		(on_board no)
+		(dnp yes)
 		(property "Reference" "H4"
 			(at 135.89 111.7599 0)
@@
 		(exclude_from_sim no)
 		(in_bom no)
-		(on_board yes)
-		(dnp no)
+		(on_board no)
+		(dnp yes)
 		(property "Reference" "H2"
 			(at 100.33 111.7599 0)
@@
 		(exclude_from_sim no)
 		(in_bom no)
-		(on_board yes)
-		(dnp no)
+		(on_board no)
+		(dnp yes)
 		(property "Reference" "H1"
 			(at 82.55 111.7599 0)
@@
 		(exclude_from_sim no)
 		(in_bom no)
-		(on_board yes)
-		(dnp no)
+		(on_board no)
+		(dnp yes)
 		(property "Reference" "H3"
 			(at 118.11 111.7599 0)

Commit message: Add pdf/
Other:
- company: (none) -> //piernov
- title: (none) -> AmbientCN3791 AnalogI2SMic
Changed lines of the file:
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@@
 	(generator_version "9.0")
 	(paper "A4")
+	(title_block
+		(title "AmbientCN3791 AnalogI2SMic")
+		(date "2025-03-04")
+		(rev "v0.1")
+		(company "//piernov")
+	)
 	(junction
 		(at 106.68 119.38)

Commit message: v0.4: Omar Titouhi 08/10/25
Other:
- added sheet Wake_Up (Wake_Up.kicad_sch)
Changed lines of the file:
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@@
+		)
+	)
+	(sheet
+		(at 208.28 53.34)
+		(size 43.18 24.13)
+		(exclude_from_sim no)
+		(in_bom yes)
+		(on_board yes)
+		(dnp no)
+		(fields_autoplaced yes)
+		(stroke
+			(width 0.1524)
+			(type solid)
+		)
+		(fill
+			(color 0 0 0 0.0000)
+		)
+		(property "Sheetname" "Wake_Up"
+			(at 208.28 52.6284 0)
+			(effects
+				(font
+					(size 1.27 1.27)
+				)
+				(justify left bottom)
+			)
+		)
+		(property "Sheetfile" "Wake_Up.kicad_sch"
+			(at 208.28 78.0546 0)
+			(effects
+				(font
+					(size 1.27 1.27)
+				)
+				(justify left top)
+			)
+		)
+		(instances
+			(project "AudioPowerBoard"
+				(path "/8cac44a1-bcd4-4356-b890-bed775abd56a"
+					(page "4")
+				)
+			)
 		)
 	)

Commit message: WIP: 0.5
Other:
- sheet Wake_Up renamed AnalogWakeUp
Changed lines of the file:
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@@
 	(title_block
 		(title "AmbientCN3791 AnalogI2SMic")
-		(date "2025-07-15")
-		(rev "v0.3")
+		(date "2026-03-11")
+		(rev "v0.5")
 		(company "//piernov")
 	)
@@
 			(color 0 0 0 0.0000)
 		)
-		(property "Sheetname" "Wake_Up"
+		(property "Sheetname" "AnalogWakeUp"
 			(at 208.28 52.6284 0)
 			(effects
